File: robot-logic-pcb.kicad_pcb (KiCad board)
At the start: 2 copper layers, 150 x 80 mm, 20 parts, among them J1 Conn_02x07_Top_Bottom, J2 Conn_01x02, J3 Conn_01x06, J4 Conn_01x06, J5 Conn_01x06, J6 Conn_01x04, J7 Conn_01x04, J8 Conn_01x04, U1 NRF24L01_Breakout

Commit message: v1
Parts:
- removed ? (x4): , 
- removed REF**: MountingHole_2.5mm, MountingHole:MountingHole_2.5mm
- A1: moved to F.Cu
- R2: value 220 -> 480
- moved J2 85.9 mm to (132.0, 78.0)
- moved A1 52.1 mm to (140.4, 50.5)
- moved J4 50.9 mm to (92.8, 93.5)
- moved U1 46.8 mm to (111.7, 59.4), turned to 0 degrees
- moved R1 46.5 mm to (128.5, 96.3), turned to 180 degrees
- moved C1 45.4 mm to (105.0, 61.5), turned to 90 degrees
- moved J6 43.2 mm to (55.5, 79.8)
- moved D1 42.9 mm to (133.7, 95.8), turned to 0 degrees
- moved J7 42.6 mm to (92.8, 66.2)
- moved J8 41.6 mm to (55.5, 91.5)
- moved R2 36.1 mm to (128.5, 86.5), turned to 180 degrees
- moved D2 34.7 mm to (133.7, 86.5), turned to 0 degrees
- moved J5 34.5 mm to (92.8, 84.0)
- moved J1 33.1 mm to (53.5, 71.5), turned to 90 degrees
- moved J3 25.2 mm to (92.8, 75.0)
Connections:
- A1 pad D13: unconnected-(A1-PadD13) -> /STATUS-LED
- A1 pad D2: /STATUS-LED -> /IRQ
- A1 pad D29: /PWR-PCB.PUMP-RLY -> unconnected-(A1-PadD29)
- A1 pad D3: /POWER-LED -> unconnected-(A1-D3_INT1-PadD3)
- A1 pad D30: /PWR-PCB.GRB-STEP -> unconnected-(A1-PadD30)
- A1 pad D31: /PWR-PCB.GRB-DIR -> unconnected-(A1-PadD31)
- A1 pad D32: /PWR-PCB.SC-STEP -> /PWR-PCB.PUMP-RLY
- A1 pad D33: /PWR-PCB.SC-DIR -> unconnected-(A1-PadD33)
- A1 pad D34: unconnected-(A1-PadD34) -> /PWR-PCB.GRB-STEP
- A1 pad D36: unconnected-(A1-PadD36) -> /PWR-PCB.GRB-DIR
- A1 pad D38: unconnected-(A1-PadD38) -> /PWR-PCB.SC-STEP
- A1 pad D4: /IRQ -> unconnected-(A1-PadD4)
- A1 pad D40: unconnected-(A1-PadD40) -> /PWR-PCB.SC-DIR
- J1 pad 1: /PWR-PCB.SBR-RX -> /PWR-PCB.PUMP-RLY
- J1 pad 10: /PWR-PCB.PUMP-RLY -> /PWR-PCB.SBR-RX
- J1 pad 2: /PWR-PCB.GRB-RX -> /PWR-PCB.GRB-TX
- J1 pad 3: /PWR-PCB.GRB-DIR -> /PWR-PCB.GRB-STEP
- J1 pad 4: /PWR-PCB.GRB-TX -> /PWR-PCB.GRB-RX
- J1 pad 5: /PWR-PCB.GRB-STEP -> /PWR-PCB.GRB-DIR
- J1 pad 6: /PWR-PCB.SC-RX -> /PWR-PCB.SC-TX
- J1 pad 7: /PWR-PCB.SC-DIR -> /PWR-PCB.SC-STEP
- J1 pad 8: /PWR-PCB.SC-TX -> /PWR-PCB.SC-RX
- J1 pad 9: /PWR-PCB.SC-STEP -> /PWR-PCB.SC-DIR
- J8 pad 3: /CTRL-RX -> /CTRL-TX
- J8 pad 4: /CTRL-TX -> /CTRL-RX
- R2 pad 2: /POWER-LED -> +9V
Routing:
- net /SDA: track 202.8 -> 52.7 mm
- net /SCL: track 203.7 -> 54.2 mm
- net /PWR-PCB.GRB-TX: track 95.0 -> 33.4 mm
- net /PWR-PCB.GRB-RX: track 92.9 -> 36.4 mm
- net /PWR-PCB.SBR-RX: track 120.4 -> 64.7 mm, vias 0 -> 1
- net /CSN: track 17.8 -> 72.9 mm
- net /SCK: track 26.6 -> 76.6 mm
- net /CE: track 17.8 -> 66.8 mm
- net /PWR-PCB.GRB-DIR: track 62.2 -> 16.4 mm
- net /PWR-PCB.PUMP-RLY: track 60.9 -> 17.5 mm
- net +9V: track 97.3 -> 54.4 mm
- net /PWR-PCB.SC-RX: track 0.00 -> 42.5 mm
- net /PWR-PCB.SC-TX: track 0.00 -> 39.5 mm
- net /MOSI: track 39.7 -> 75.8 mm, vias 0 -> 1
- net /IRQ: track 82.3 -> 50.7 mm
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Other:
- board size 150 x 80 mm -> 100 x 54.3 mm
- board text added: "CTRL"
- board text added: "DIGIT"
- board text added: "FAILURE"
- board text added: "Game Team"
- board text added: "LCD"
- board text added: "LOGICAL PCB"
- board text added: "NOTICE : Input : +9V 0.2A Source : https://github.com/ Game-Team-SLSC/robot- logical-pcb-2025 Do not link front and back faces !"
- board text added: "PCA9685"
- board text added: "POWER"
- board text added: "POWER PCB"
- board text added: "VL53L0X-L"
- board text added: "VL53L0X-R"
