File: robot-logic-pcb.kicad_sch (KiCad schematic)
At the start: 15 parts, among them J1 Conn_02x07_Top_Bottom, J2 Conn_01x02, J3 Conn_01x06, J4 Conn_01x06, J5 Conn_01x06, J6 Conn_01x04, J7 Conn_01x04, J8 Conn_01x04, U1 NRF24L01_Breakout

Commit message: v1
Parts:
- R2: value 220 -> 480
Connections:
- net +9V: now also R2.2
- net CTRL-RX: now also J8.4 (Pin_4); no longer J8.3 (Pin_3)
- net CTRL-TX: now also J8.3 (Pin_3); no longer J8.4 (Pin_4)
- net IRQ: now also A1.D2 (D2_INT0); no longer A1.D4
- net PWR-PCB.GRB-DIR: now also A1.D36, J1.5 (Pin_5); no longer A1.D31, J1.3 (Pin_3)
- net PWR-PCB.GRB-RX: now also J1.4 (Pin_4); no longer J1.2 (Pin_2)
- net PWR-PCB.GRB-STEP: now also A1.D34, J1.3 (Pin_3); no longer A1.D30, J1.5 (Pin_5)
- net PWR-PCB.GRB-TX: now also J1.2 (Pin_2); no longer J1.4 (Pin_4)
- net PWR-PCB.PUMP-RLY: now also A1.D32, J1.1 (Pin_1); no longer A1.D29, J1.10 (Pin_10)
- net PWR-PCB.SBR-RX: now also J1.10 (Pin_10); no longer J1.1 (Pin_1)
- net PWR-PCB.SC-DIR: now also A1.D40, J1.9 (Pin_9); no longer A1.D33, J1.7 (Pin_7)
- net PWR-PCB.SC-RX: now also J1.8 (Pin_8); no longer J1.6 (Pin_6)
- net PWR-PCB.SC-STEP: now also A1.D38, J1.7 (Pin_7); no longer A1.D32, J1.9 (Pin_9)
- net PWR-PCB.SC-TX: now also J1.6 (Pin_6); no longer J1.8 (Pin_8)
- net STATUS-LED: now also A1.D13; no longer A1.D2 (D2_INT0)
- net POWER-LED: no longer names the net of A1.D3 (D3_INT1)
- net POWER-LED: no longer R2.2
- no-connect marks 74 -> 75
